File: peatPellet3.kicad_sch (KiCad schematic)
At the start: 56 parts, among them J1 Barrel_Jack_Switch, J2 AudioJack2, J3 AudioJack2, K1 Relay_DPDT, SW1 SW_SPDT, SW2 SW_SPDT, SW3 SW_SPDT_MSM, U1 TL072, U2 L78L05_SO8, U3 LM555xM

Commit message: end of 8/24
Parts:
- C11, C12: value C_Polarized -> XXX
Connections:
- net EXP: now also A1.5 (SD_DATA_0); no longer A1.25 (ADC_3)
- net KNOB1: now also A1.4 (SD_DATA_1); no longer A1.22 (ADC_0)
- net KNOB2: now also A1.3 (SD_DATA_2); no longer A1.23 (ADC_1)
- net KNOB3: now also A1.2 (SD_DATA_3); no longer A1.24 (ADC_2)
- net SW1: now also A1.34 (SAI2_FS); no longer A1.32 (SAI2_SD_B)
- net SW2: now also A1.35 (SAI2_SCK); no longer A1.33 (SAI2_SD_A)
- net SW3: now also A1.10 (SPI1_POCI); no longer A1.11 (SPI1_PICO)
- net SW4: now also A1.11 (SPI1_PICO); no longer A1.10 (SPI1_POCI)
- net XFS: now also A1.6 (SD_CMD); no longer A1.9 (SPI1_SCK)
Changed lines of the file:
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@@
+    (stroke (width 0) (type default))
+  )
+  (wire (pts (xy 31.75 85.09) (xy 35.56 85.09))
     (stroke (width 0) (type default))
   )
@@
     (stroke (width 0) (type default))
   )
-  (wire (pts (xy 88.9 74.93) (xy 86.36 74.93))
-    (stroke (width 0) (type default))
-  )
   (wire (pts (xy 186.69 57.15) (xy 166.37 57.15))
     (stroke (width 0) (type default))
@@
     (stroke (width 0) (type default))
   )
+  (wire (pts (xy 25.4 90.17) (xy 35.56 90.17))
+    (stroke (width 0) (type default))
+  )
   (wire (pts (xy 224.79 21.59) (xy 217.17 21.59))
     (stroke (width 0) (type default))
@@
     (stroke (width 0) (type default))
   )
+  (wire (pts (xy 25.4 95.25) (xy 35.56 95.25))
+    (stroke (width 0) (type default))
+  )
   (wire (pts (xy 231.14 76.2) (xy 227.33 76.2))
     (stroke (width 0) (type default))
@@
     (stroke (width 0) (type default))
   )
+  (wire (pts (xy 25.4 100.33) (xy 35.56 100.33))
+    (stroke (width 0) (type default))
+  )
   (wire (pts (xy 199.39 105.41) (xy 215.9 105.41))
     (stroke (width 0) (type default))
@@
     (stroke (width 0) (type default))
   )
-  (wire (pts (xy 99.06 67.31) (xy 86.36 67.31))
-    (stroke (width 0) (type default))
-  )
   (wire (pts (xy 154.94 100.33) (xy 166.37 100.33))
     (stroke (width 0) (type default))
@@
     (stroke (width 0) (type default))
   )
+  (wire (pts (xy 24.13 82.55) (xy 35.56 82.55))
+    (stroke (width 0) (type default))
+  )
   (wire (pts (xy 215.9 110.49) (xy 212.09 110.49))
     (stroke (width 0) (type default))
@@
     (stroke (width 0) (type default))
   )
-  (wire (pts (xy 35.56 85.09) (xy 24.13 85.09))
-    (stroke (width 0) (type default))
-  )
   (wire (pts (xy 146.05 58.42) (xy 146.05 62.23))
     (stroke (width 0) (type default))
@@
     (stroke (width 0) (type default))
   )
-  (wire (pts (xy 35.56 80.01) (xy 24.13 80.01))
-    (stroke (width 0) (type default))
-  )
   (wire (pts (xy 170.18 92.71) (xy 189.23 92.71))
     (stroke (width 0) (type default))
@@
     (stroke (width 0) (type default))
   )
+  (wire (pts (xy 86.36 100.33) (xy 88.9 100.33))
+    (stroke (width 0) (type default))
+  )
   (wire (pts (xy 60.96 31.75) (xy 60.96 39.37))
     (stroke (width 0) (type default))
@@
     (stroke (width 0) (type default))
   )
-  (wire (pts (xy 88.9 69.85) (xy 86.36 69.85))
-    (stroke (width 0) (type default))
-  )
-  (wire (pts (xy 97.79 97.79) (xy 86.36 97.79))
-    (stroke (width 0) (type default))
-  )
   (wire (pts (xy 242.57 40.64) (xy 242.57 44.45))
     (stroke (width 0) (type default))
@@
     (stroke (width 0) (type default))
   )
-  (wire (pts (xy 91.44 95.25) (xy 86.36 95.25))
-    (stroke (width 0) (type default))
-  )
   (wire (pts (xy 222.25 128.27) (xy 222.25 134.62))
     (stroke (width 0) (type default))
@@
     (stroke (width 0) (type default))
   )
+  (wire (pts (xy 86.36 102.87) (xy 95.25 102.87))
+    (stroke (width 0) (type default))
+  )
   (wire (pts (xy 224.79 41.91) (xy 219.71 41.91))
     (stroke (width 0) (type default))
@@
     (stroke (width 0) (type default))
   )
+  (wire (pts (xy 34.29 92.71) (xy 35.56 92.71))
+    (stroke (width 0) (type default))
+  )
   (wire (pts (xy 121.92 107.95) (xy 134.62 107.95))
     (stroke (width 0) (type default))
@@
     (stroke (width 0) (type default))
   )
-  (wire (pts (xy 97.79 72.39) (xy 86.36 72.39))
-    (stroke (width 0) (type default))
-  )
   (wire (pts (xy 113.03 48.26) (xy 113.03 17.78))
     (stroke (width 0) (type default))
@@
     (stroke (width 0) (type default))
   )
-  (wire (pts (xy 35.56 82.55) (xy 31.75 82.55))
+  (wire (pts (xy 34.29 97.79) (xy 35.56 97.79))
     (stroke (width 0) (type default))
   )
@@
     )
   )
-  (global_label "SW4" (shape passive) (at 31.75 82.55 180) (fields_autoplaced)
+  (global_label "SW4" (shape passive) (at 31.75 85.09 180) (fields_autoplaced)
     (effects (font (size 1.27 1.27)) (justify right))
-    (property "Intersheetrefs" "${INTERSHEET_REFS}" (at 26.0057 82.55 0)
+    (property "Intersheetrefs" "${INTERSHEET_REFS}" (at 26.0057 85.09 0)
       (effects (font (size 1.27 1.27)) (justify right) hide)
     )
@@
     )
   )
-  (global_label "SW2" (shape passive) (at 97.79 97.79 0) (fields_autoplaced)
+  (global_label "SW2" (shape passive) (at 95.25 102.87 0) (fields_autoplaced)
     (effects (font (size 1.27 1.27)) (justify left))
-    (property "Intersheetrefs" "${INTERSHEET_REFS}" (at 103.5343 97.79 0)
+    (property "Intersheetrefs" "${INTERSHEET_REFS}" (at 100.9943 102.87 0)
       (effects (font (size 1.27 1.27)) (justify left) hide)
     )
@@
     )
   )
-  (global_label "KNOB2" (shape passive) (at 88.9 69.85 0) (fields_autoplaced)
-    (effects (font (size 1.27 1.27)) (justify left))
-    (property "Intersheetrefs" "${INTERSHEET_REFS}" (at 97.1844 69.85 0)
-      (effects (font (size 1.27 1.27)) (justify left) hide)
+  (global_label "KNOB2" (shape passive) (at 25.4 95.25 180) (fields_autoplaced)
+    (effects (font (size 1.27 1.27)) (justify right))
+    (property "Intersheetrefs" "${INTERSHEET_REFS}" (at 17.1156 95.25 0)
+      (effects (font (size 1.27 1.27)) (justify right) hide)
     )
   )
@@
     )
   )
-  (global_label "KNOB1" (shape passive) (at 99.06 67.31 0) (fields_autoplaced)
-    (effects (font (size 1.27 1.27)) (justify left))
-    (property "Intersheetrefs" "${INTERSHEET_REFS}" (at 107.3444 67.31 0)
-      (effects (font (size 1.27 1.27)) (justify left) hide)
+  (global_label "KNOB1" (shape passive) (at 34.29 92.71 180) (fields_autoplaced)
+    (effects (font (size 1.27 1.27)) (justify right))
+    (property "Intersheetrefs" "${INTERSHEET_REFS}" (at 26.0056 92.71 0)
+      (effects (font (size 1.27 1.27)) (justify right) hide)
     )
   )
@@
     )
   )
-  (global_label "SW1" (shape passive) (at 91.44 95.25 0) (fields_autoplaced)
+  (global_label "SW1" (shape passive) (at 88.9 100.33 0) (fields_autoplaced)
     (effects (font (size 1.27 1.27)) (justify left))
-    (property "Intersheetrefs" "${INTERSHEET_REFS}" (at 97.1843 95.25 0)
+    (property "Intersheetrefs" "${INTERSHEET_REFS}" (at 94.6443 100.33 0)
       (effects (font (size 1.27 1.27)) (justify left) hide)
     )
@@
     )
   )
-  (global_label "SW3" (shape passive) (at 24.13 85.09 180) (fields_autoplaced)
+  (global_label "SW3" (shape passive) (at 24.13 82.55 180) (fields_autoplaced)
     (effects (font (size 1.27 1.27)) (justify right))
-    (property "Intersheetrefs" "${INTERSHEET_REFS}" (at 18.3857 85.09 0)
+    (property "Intersheetrefs" "${INTERSHEET_REFS}" (at 18.3857 82.55 0)
       (effects (font (size 1.27 1.27)) (justify right) hide)
     )
@@
     )
   )
-  (global_label "KNOB3" (shape passive) (at 97.79 72.39 0) (fields_autoplaced)
-    (effects (font (size 1.27 1.27)) (justify left))
-    (property "Intersheetrefs" "${INTERSHEET_REFS}" (at 106.0744 72.39 0)
-      (effects (font (size 1.27 1.27)) (justify left) hide)
+  (global_label "KNOB3" (shape passive) (at 34.29 97.79 180) (fields_autoplaced)
+    (effects (font (size 1.27 1.27)) (justify right))
+    (property "Intersheetrefs" "${INTERSHEET_REFS}" (at 26.0056 97.79 0)
+      (effects (font (size 1.27 1.27)) (justify right) hide)
     )
   )
@@
     )
   )
-  (global_label "XFS" (shape passive) (at 24.13 80.01 180) (fields_autoplaced)
+  (global_label "XFS" (shape passive) (at 25.4 100.33 180) (fields_autoplaced)
     (effects (font (size 1.27 1.27)) (justify right))
-    (property "Intersheetrefs" "${INTERSHEET_REFS}" (at 18.7485 80.01 0)
+    (property "Intersheetrefs" "${INTERSHEET_REFS}" (at 20.0185 100.33 0)
       (effects (font (size 1.27 1.27)) (justify right) hide)
     )
@@
     )
   )
-  (global_label "EXP" (shape passive) (at 88.9 74.93 0) (fields_autoplaced)
-    (effects (font (size 1.27 1.27)) (justify left))
-    (property "Intersheetrefs" "${INTERSHEET_REFS}" (at 94.4024 74.93 0)
-      (effects (font (size 1.27 1.27)) (justify left) hide)
+  (global_label "EXP" (shape passive) (at 25.4 90.17 180) (fields_autoplaced)
+    (effects (font (size 1.27 1.27)) (justify right))
+    (property "Intersheetrefs" "${INTERSHEET_REFS}" (at 19.8976 90.17 0)
+      (effects (font (size 1.27 1.27)) (justify right) hide)
     )
   )
@@
       (effects (font (size 1.27 1.27)) (justify left))
     )
-    (property "Value" "C_Polarized" (at 185.42 114.681 0)
+    (property "Value" "XXX" (at 185.42 114.681 0)
       (effects (font (size 1.27 1.27)) (justify left))
     )
@@
       (effects (font (size 1.27 1.27)) (justify left))
     )
-    (property "Value" "C_Polarized" (at 138.43 127.381 0)
-      (effects (font (size 1.27 1.27)) (justify left))
-    )
+    (property "Value" "XXX" (at 138.43 127.381 0)
+      (effects (font (size 1.27 1.27)) (justify left))
+    )
