File: peatPellet3.kicad_pcb (KiCad board)
At the start: 2 copper layers, 87.6 x 56.5 mm, 63 parts, among them J1 Barrel_Jack_Switch, J2 AudioJack2, J3 AudioJack2, K1 Relay_DPDT, SW1 SW_SPDT, SW2 SW_SPDT, SW3 SW_SPDT_MSM, U1 TL072, U2 L78L05_SO8, U3 LM555xM

Commit message: footprint shifts
Parts:
- moved ? 3.86 mm to (73.7, 130.1)
- moved R11 1.39 mm to (104.8, 104.8)
- moved R12 0.27 mm to (104.8, 102.9)
Routing:
- net Net-(C12-Pad1): track 12.1 -> 20.1 mm
- net Net-(U3-THR): track 34.8 -> 34.3 mm
Changed lines of the file:
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@@
   )
   (footprint "Resistor_SMD:R_0603_1608Metric" (layer "F.Cu")
-    (at 105.345 106.045 180)
+    (at 104.785 104.775 180)
     (descr "Resistor SMD 0603 (1608 Metric), square (rectangular) end terminal, IPC_7351 nominal, (Body size source: IPC-SM-782 page 72, https://www.pcb-3d.com/wordpress/wp-content/uploads/ipc-sm-782a_amendment_1_and_2.pdf), generated with kicad-footprint-generator")
     (tags "resistor")
@@
   )
   (footprint "enclosures:MOMENTARY" (layer "F.Cu")
-    (at 69.85 130.712501 -90)
+    (at 73.66 130.077501 -90)
     (attr through_hole)
     (fp_text reference "" (at 0 0 -270) (layer "F.SilkS")
@@
   )
   (footprint "Resistor_SMD:R_0603_1608Metric" (layer "F.Cu")
-    (at 104.52 102.87 180)
+    (at 104.785 102.87 180)
     (descr "Resistor SMD 0603 (1608 Metric), square (rectangular) end terminal, IPC_7351 nominal, (Body size source: IPC-SM-782 page 72, https://www.pcb-3d.com/wordpress/wp-content/uploads/ipc-sm-782a_amendment_1_and_2.pdf), generated with kicad-footprint-generator")
     (tags "resistor")
@@
   (segment (start 101.155 118.555) (end 100.965 118.745) (width 0.25) (layer "F.Cu") (net 17))
   (segment (start 101.5105 112.03) (end 100.965 112.5755) (width 0.25) (layer "F.Cu") (net 17))
-  (segment (start 106.045 99.06) (end 106.045 99.1495) (width 0.25) (layer "F.Cu") (net 17))
   (segment (start 135.89 135.89) (end 135.89 137.3) (width 0.25) (layer "F.Cu") (net 17))
   (segment (start 92.205 117.98) (end 91.44 118.745) (width 0.25) (layer "F.Cu") (net 17))
@@
   (segment (start 99.695 104.14) (end 98.425 105.41) (width 0.25) (layer "F.Cu") (net 17))
   (segment (start 88.075 116.255) (end 88.125 116.205) (width 0.25) (layer "F.Cu") (net 17))
-  (segment (start 107.315 100.33) (end 106.045 99.06) (width 0.25) (layer "F.Cu") (net 17))
   (segment (start 102.235 100.965) (end 101.6 100.33) (width 0.25) (layer "F.Cu") (net 17))
   (segment (start 123.19 104.47) (end 123.19 105.41) (width 0.25) (layer "F.Cu") (net 17))
   (segment (start 104.905 114.935) (end 104.905 116.205) (width 0.25) (layer "F.Cu") (net 17))
+  (segment (start 109.855 100.33) (end 107.76 100.33) (width 0.25) (layer "F.Cu") (net 17))
   (segment (start 104.905 114.935) (end 105.281751 114.935) (width 0.25) (layer "F.Cu") (net 17))
   (segment (start 105.281751 114.935) (end 106.68 113.536751) (width 0.25) (layer "F.Cu") (net 17))
@@
   (segment (start 104.88 111.23) (end 103.53 111.23) (width 0.25) (layer "F.Cu") (net 17))
   (segment (start 100.4195 112.03) (end 100.965 112.5755) (width 0.25) (layer "F.Cu") (net 17))
-  (segment (start 107.76 100.33) (end 107.315 100.33) (width 0.25) (layer "F.Cu") (net 17))
   (segment (start 112.04 111.76) (end 113.665 111.76) (width 0.25) (layer "F.Cu") (net 17))
   (segment (start 99.34 112.03) (end 100.4195 112.03) (width 0.25) (layer "F.Cu") (net 17))
@@
   (via (at 100.965 118.745) (size 0.8) (drill 0.4) (layers "F.Cu" "B.Cu") (net 17))
   (via (at 100.965 112.5755) (size 0.8) (drill 0.4) (layers "F.Cu" "B.Cu") (net 17))
-  (via (at 106.045 99.1495) (size 0.8) (drill 0.4) (layers "F.Cu" "B.Cu") (net 17))
+  (via (at 109.855 100.33) (size 0.8) (drill 0.4) (layers "F.Cu" "B.Cu") (net 17))
   (via (at 92.71 106.315) (size 0.8) (drill 0.4) (layers "F.Cu" "B.Cu") (net 17))
   (via (at 123.19 105.41) (size 0.8) (drill 0.4) (layers "F.Cu" "B.Cu") (net 17))
@@
   (segment (start 104.905 113.665) (end 104.905 112.655) (width 0.25) (layer "F.Cu") (net 45))
   (segment (start 107.76 101.6) (end 106.68 101.6) (width 0.25) (layer "F.Cu") (net 48))
-  (segment (start 104.52 100.965) (end 104.52 104.14) (width 0.25) (layer "F.Cu") (net 48))
-  (segment (start 104.52 106.045) (end 104.52 104.14) (width 0.25) (layer "F.Cu") (net 48))
-  (segment (start 103.747538 104.14) (end 104.52 104.14) (width 0.25) (layer "F.Cu") (net 48))
-  (segment (start 98.425 98.817462) (end 103.747538 104.14) (width 0.25) (layer "F.Cu") (net 48))
-  (segment (start 106.035 103.515) (end 105.41 104.14) (width 0.25) (layer "F.Cu") (net 48))
+  (segment (start 104.52 100.965) (end 104.685 101.13) (width 0.25) (layer "F.Cu") (net 48))
+  (segment (start 98.425 98.817462) (end 103.400787 103.793249) (width 0.25) (layer "F.Cu") (net 48))
+  (segment (start 106.391751 103.793249) (end 105.41 103.793249) (width 0.25) (layer "F.Cu") (net 48))
+  (segment (start 106.69 103.495) (end 106.391751 103.793249) (width 0.25) (layer "F.Cu") (net 48))
+  (segment (start 104.685 103.536498) (end 104.941751 103.793249) (width 0.25) (layer "F.Cu") (net 48))
   (segment (start 99.695 90.17) (end 98.425 91.44) (width 0.25) (layer "F.Cu") (net 48))
-  (segment (start 105.41 104.14) (end 104.52 104.14) (width 0.25) (layer "F.Cu") (net 48))
+  (segment (start 103.400787 103.793249) (end 105.41 103.793249) (width 0.25) (layer "F.Cu") (net 48))
+  (segment (start 112.71 102.87) (end 112.085 103.495) (width 0.25) (layer "F.Cu") (net 48))
+  (segment (start 105.41 103.793249) (end 104.941751 103.793249) (width 0.25) (layer "F.Cu") (net 48))
+  (segment (start 104.685 101.13) (end 104.685 103.536498) (width 0.25) (layer "F.Cu") (net 48))
   (segment (start 106.045 100.965) (end 104.52 100.965) (width 0.25) (layer "F.Cu") (net 48))
-  (segment (start 112.71 102.87) (end 112.065 103.515) (width 0.25) (layer "F.Cu") (net 48))
   (segment (start 106.68 101.6) (end 106.045 100.965) (width 0.25) (layer "F.Cu") (net 48))
-  (segment (start 112.065 103.515) (end 106.035 103.515) (width 0.25) (layer "F.Cu") (net 48))
+  (segment (start 112.085 103.495) (end 106.69 103.495) (width 0.25) (layer "F.Cu") (net 48))
   (segment (start 98.425 91.44) (end 98.425 98.817462) (width 0.25) (layer "F.Cu") (net 48))
+  (segment (start 104.941751 103.793249) (end 103.96 104.775) (width 0.25) (layer "F.Cu") (net 48))
   (segment (start 89.945 110.71) (end 89.725 110.49) (width 0.25) (layer "F.Cu") (net 51))
   (segment (start 88.655 97.73) (end 89.535 96.85) (width 0.25) (layer "F.Cu") (net 51))
@@
   (segment (start 93.855 110.49) (end 93.855 109.235) (width 0.25) (layer "F.Cu") (net 53))
   (segment (start 93.855 109.235) (end 93.205 108.585) (width 0.25) (layer "F.Cu") (net 53))
-  (segment (start 103.695 102.87) (end 103.695 90.805) (width 0.25) (layer "F.Cu") (net 54))
+  (segment (start 98.496 88.829) (end 101.719 88.829) (width 0.25) (layer "F.Cu") (net 54))
+  (segment (start 103.695 90.805) (end 103.695 102.605) (width 0.25) (layer "F.Cu") (net 54))
+  (segment (start 103.695 102.605) (end 103.96 102.87) (width 0.25) (layer "F.Cu") (net 54))
+  (segment (start 101.719 88.829) (end 103.695 90.805) (width 0.25) (layer "F.Cu") (net 54))
+  (segment (start 97.155 90.17) (end 98.496 88.829) (width 0.25) (layer "F.Cu") (net 54))
   (segment (start 115.695 96.4) (end 115.565 96.27) (width 0.25) (layer "F.Cu") (net 55))
   (segment (start 115.565 96.27) (end 115.565 92.075) (width 0.25) (layer "F.Cu") (net 55))
@@
   (segment (start 157.48 130.175) (end 157.48 128.905) (width 0.25) (layer "F.Cu") (net 65))
   (segment (start 114.755 104.765) (end 116.32 103.2) (width 0.25) (layer "F.Cu") (net 66))
-  (segment (start 107.76 104.455) (end 107.76 104.14) (width 0.25) (layer "F.Cu") (net 66))
   (segment (start 112.71 100.33) (end 115.825 100.33) (width 0.25) (layer "F.Cu") (net 66))
   (segment (start 125.095 104.52) (end 125.095 107.835) (width 0.25) (layer "F.Cu") (net 66))
@@
   (segment (start 125.095 107.835) (end 122.44 110.49) (width 0.25) (layer "F.Cu") (net 66))
   (segment (start 115.825 102.705) (end 116.32 103.2) (width 0.25) (layer "F.Cu") (net 66))
+  (segment (start 107.125 104.775) (end 107.76 104.14) (width 0.25) (layer "F.Cu") (net 66))
   (segment (start 115.825 100.33) (end 115.825 102.705) (width 0.25) (layer "F.Cu") (net 66))
-  (segment (start 106.17 106.045) (end 107.76 104.455) (width 0.25) (layer "F.Cu") (net 66))
   (segment (start 122.32 122.851701) (end 123.293299 123.825) (width 0.25) (layer "F.Cu") (net 66))
   (segment (start 134.34 137.3) (end 133.845 137.795) (width 0.25) (layer "F.Cu") (net 66))
   (segment (start 123.293299 123.825) (end 127.635 123.825) (width 0.25) (layer "F.Cu") (net 66))
+  (segment (start 105.61 104.775) (end 107.125 104.775) (width 0.25) (layer "F.Cu") (net 66))
   (segment (start 134.34 135.89) (end 134.34 137.3) (width 0.25) (layer "F.Cu") (net 66))
   (segment (start 123.075 110.49) (end 124.588 112.003) (width 0.25) (layer "F.Cu") (net 66))
