File: peatPellet3.kicad_pcb (KiCad board)
At the start: 2 copper layers, 87.6 x 56.5 mm, 63 parts, among them J1 Barrel_Jack_Switch, J2 AudioJack2, J3 AudioJack2, K1 Relay_DPDT, SW1 SW_SPDT, SW2 SW_SPDT, SW3 SW_SPDT_MSM, U1 TL072, U2 L78L05_SO8, U3 LM555xM

Commit message: via cleanup
Parts:
- moved C3 1.65 mm to (112.9, 112.0)
- moved R10 1.09 mm to (104.8, 101.0)
- moved R14 0.52 mm to (103.2, 98.4)
- moved R11 0.38 mm to (104.8, 104.4)
- moved R12 0.37 mm to (104.8, 102.5)
- moved D5 0.30 mm to (104.1, 96.5)
Routing:
- net Net-(D4-A): track 4.36 -> 12.4 mm
- net GND: track 49.7 -> 42.3 mm
- net Net-(U3-THR): track 34.3 -> 31.9 mm
- net +9V: track 66.5 -> 64.2 mm
- net Net-(D4-K): track 6.23 -> 6.78 mm

Commit message: via update 2
Routing:
- net GND: track 42.3 -> 46.5 mm
Changed lines of the file:
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@@
   (segment (start 88.075 117.7925) (end 88.075 116.84) (width 0.25) (layer "F.Cu") (net 17))
   (segment (start 120.015 104.775) (end 121.59 103.2) (width 0.25) (layer "F.Cu") (net 17))
-  (segment (start 93.855 106.68) (end 93.075 106.68) (width 0.25) (layer "F.Cu") (net 17))
   (segment (start 104.265 96.52) (end 105.535 96.52) (width 0.25) (layer "F.Cu") (net 17))
   (segment (start 103.53 111.23) (end 102.73 112.03) (width 0.25) (layer "F.Cu") (net 17))
   (segment (start 113.025 92.075) (end 110.565 92.075) (width 0.25) (layer "F.Cu") (net 17))
-  (segment (start 93.075 106.68) (end 92.71 106.315) (width 0.25) (layer "F.Cu") (net 17))
   (segment (start 106.68 113.536751) (end 106.68 113.03) (width 0.25) (layer "F.Cu") (net 17))
   (segment (start 86.8 117.05) (end 87.865 117.05) (width 0.25) (layer "F.Cu") (net 17))
@@
   (segment (start 104.775 100.15) (end 103.96 100.965) (width 0.25) (layer "F.Cu") (net 17))
   (segment (start 115.57 112.03) (end 116.84 110.76) (width 0.25) (layer "F.Cu") (net 17))
+  (segment (start 109.855 114.935) (end 107.95 114.935) (width 0.25) (layer "F.Cu") (net 17))
+  (segment (start 106.68 113.665) (end 106.68 113.03) (width 0.25) (layer "F.Cu") (net 17))
   (segment (start 104.905 114.935) (end 104.905 116.205) (width 0.25) (layer "F.Cu") (net 17))
   (segment (start 109.855 100.33) (end 107.76 100.33) (width 0.25) (layer "F.Cu") (net 17))
@@
   (segment (start 104.88 111.23) (end 103.53 111.23) (width 0.25) (layer "F.Cu") (net 17))
   (segment (start 93.8905 117.475) (end 92.205 117.475) (width 0.25) (layer "F.Cu") (net 17))
+  (segment (start 107.95 114.935) (end 106.68 113.665) (width 0.25) (layer "F.Cu") (net 17))
   (segment (start 113.665 112.03) (end 115.57 112.03) (width 0.25) (layer "F.Cu") (net 17))
   (segment (start 110.565 92.075) (end 109.295 90.805) (width 0.25) (layer "F.Cu") (net 17))
+  (segment (start 93.855 106.68) (end 92.71 106.68) (width 0.25) (layer "F.Cu") (net 17))
   (segment (start 104.775 99.695) (end 104.775 100.15) (width 0.25) (layer "F.Cu") (net 17))
   (segment (start 109.855 114.935) (end 109.855 116.205) (width 0.25) (layer "F.Cu") (net 17))
@@
   (via (at 101.05 112.03) (size 0.8) (drill 0.4) (layers "F.Cu" "B.Cu") (net 17))
   (via (at 109.855 100.33) (size 0.8) (drill 0.4) (layers "F.Cu" "B.Cu") (net 17))
-  (via (at 92.71 106.315) (size 0.8) (drill 0.4) (layers "F.Cu" "B.Cu") (net 17))
+  (via (at 92.71 106.68) (size 0.8) (drill 0.4) (layers "F.Cu" "B.Cu") (net 17))
   (via (at 104.775 99.695) (size 0.8) (drill 0.4) (layers "F.Cu" "B.Cu") (net 17))
   (via (at 120.015 104.775) (size 0.8) (drill 0.4) (layers "F.Cu" "B.Cu") (net 17))

Commit message: updated pcb layou
Parts:
- moved C3 1.77 mm to (111.1, 112.0)
- moved R17 1.37 mm to (154.1, 133.9)
- moved R15 0.68 mm to (116.3, 133.9)
- moved R9 0.53 mm to (108.3, 133.9)
- moved C1 0.52 mm to (119.1, 110.5)
- moved R16 0.46 mm to (124.3, 133.9)
- moved D10 0.25 mm to (154.9, 129.2)
- moved D7 0.25 mm to (109.1, 129.2)
- moved D8 0.25 mm to (117.1, 129.2)
- moved D9 0.25 mm to (125.1, 129.2)
Routing:
- net GND: track 46.5 -> 43.0 mm, vias 12 -> 13
- net +9V: track 64.2 -> 66.1 mm
- net LED5: track 45.5 -> 46.6 mm
- net Net-(D10-A): track 6.39 -> 5.76 mm
- net LED3: track 10.6 -> 11.2 mm
